File: Kicad/ReflowOven.kicad_pcb (KiCad board)
At the start: 2 copper layers, 48.7 x 48.9 mm, 21 parts, among them J1 Relay_Conn, P1 USB_B, SW1 Reset, SW2 TEST_SW, U1 AD595AQ, U2 AT90USB646-MU, Y1 16Mhz

Commit message: Update
Parts:
- added GS1: GS2, Connectors:GS2, F.Cu at (101.9, 100.8)
- added GS3: GS4, Connectors:GS2, F.Cu at (134.9, 90.4)
- added P2: HE10-10, .pretty:he10-10d, F.Cu at (137.1, 112.7)
- added Q1: BC817-40, TO_SOT_Packages_SMD:SOT-23, F.Cu at (141.2, 115.6)
- added R4: 1k, Resistors_SMD:R_0805_HandSoldering, F.Cu at (135.8, 95.6)
- added R5: 1k, Resistors_SMD:R_0805_HandSoldering, F.Cu at (135.8, 97.6)
- added R6: 1k, Resistors_SMD:R_0805_HandSoldering, F.Cu at (135.8, 99.4)
- added R7: 1k, Resistors_SMD:R_0805_HandSoldering, F.Cu at (140.4, 101.2)
- added R8: 1k, Resistors_SMD:R_0805_HandSoldering, F.Cu at (135.7, 114.7)
- ?: renamed from REF***; footprint Symbols:KiCad-Logo2_8mm_SilkScreen -> Symbols:Symbol_GNU-Logo_CopperTop
- ?: renamed from REF***; footprint Symbols:OSHW-Logo2_9.8x8mm_SilkScreen -> Symbols:OSHW-Logo_11.4x12mm_Copper
- C2, C3: value 22pf -> 10pf
- P1: value USB_B -> USB_OTG; footprint Connectors:USB_A -> fmcw2_mcu:USB_MICRO
- R1: value 1M -> 1k
- moved R1 21.4 mm to (106.9, 100.7), turned to 90 degrees
- moved J1 10.1 mm to (145.1, 110.4)
- moved D4 7.57 mm to (145.0, 101.2)
- moved ? 6.89 mm to (139.6, 126.7)
- moved D2 6.12 mm to (140.3, 96.1), turned to 180 degrees
- moved ? 4.82 mm to (101.4, 125.6)
- moved D5 4.46 mm to (140.4, 99.4), turned to 180 degrees
- moved P1 4.07 mm to (98.6, 106.6)
- moved D3 4.02 mm to (140.4, 97.8), turned to 180 degrees
- moved D1 3.44 mm to (109.2, 98.1)
Connections:
- D1 pad 2: /VBUS -> Net-(D1-Pad2)
- D2 pad 2: /PA0_TEST_IC -> Net-(D2-Pad2)
- D3 pad 2: /PA1_PRE_HEAT -> Net-(D3-Pad2)
- D4 pad 2: /PA3_COOL -> Net-(D4-Pad2)
- D5 pad 2: /PA2_REFLOW -> Net-(D5-Pad2)
- J1 pad 1: /Relay+ -> Net-(J1-Pad1)
- J1 pad 2: /Relay- -> /VBUS
- P1 pad 4: GND -> Net-(P1-Pad4)
- R1 pad 1: Net-(C2-Pad1) -> /VBUS
- R1 pad 2: Net-(C3-Pad1) -> Net-(D1-Pad2)
- U2 pad 35: /Relay+ -> /Relay
- U2 pad 36: /Relay- -> Net-(U2-Pad36)
- U2 pad 43: Net-(U2-Pad43) -> /HWB
Routing:
- net GND: track 183.0 -> 229.1 mm
- net /VBUS: track 56.7 -> 92.8 mm
- net /Relay-: track 10.4 -> 0.00 mm
- net /Relay+: track 10.4 -> 0.00 mm
- net Net-(P2-Pad1): track 0.00 -> 9.50 mm
- net Net-(P2-Pad3): track 0.00 -> 8.79 mm
- net /HWB: track 0.00 -> 8.75 mm
- net Net-(P2-Pad7): track 0.00 -> 8.34 mm
- net Net-(P2-Pad9): track 0.00 -> 7.95 mm
- net Net-(P2-Pad2): track 0.00 -> 7.21 mm
- net /PA2_REFLOW: track 13.6 -> 6.95 mm
- net /Relay: track 0.00 -> 6.51 mm
- net Net-(J1-Pad1): track 0.00 -> 6.39 mm
- net Net-(P2-Pad4): track 0.00 -> 5.92 mm
- net Net-(P2-Pad6): track 0.00 -> 5.53 mm
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Other:
- board size 48.7 x 48.9 mm -> 57.5 x 48.9 mm

Commit message: Modified Files
Parts:
- removed C3: 10pf, Capacitors_SMD:C_0805_HandSoldering
- added ?: KiCad-Logo2_6mm_SilkScreen, Symbols:KiCad-Logo2_6mm_SilkScreen, F.Cu at (121.2, 128.9)
- added ?: Symbol_GNU-Logo_SilkscreenTop, Symbols:Symbol_GNU-Logo_SilkscreenTop, F.Cu at (101.4, 125.7)
- added ?: OSHW-Logo_11.4x12mm_SilkScreen, Symbols:OSHW-Logo_11.4x12mm_SilkScreen, F.Cu at (139.5, 126.8)
- added R10: 24k, Resistors_SMD:R_0805_HandSoldering, F.Cu at (118.7, 122.4)
- added R9: 12k, Resistors_SMD:R_0805_HandSoldering, F.Cu at (117.2, 118.7)
- C1: value 2.2uf -> 10uf
- C2: value 10pf -> 0.01uf
- Y1: footprint Crystals:Crystal_AT310_d3.0mm_l10.0mm_Horizontal -> Crystals:Crystal_SMD_3225-4pin_3.2x2.5mm_HandSoldering
- moved C2 7.46 mm to (123.6, 122.4), turned to 180 degrees
- moved Y1 1.67 mm to (121.7, 118.7)
- renumbered P2 to ?
Connections:
- C2 pad 1: Net-(C2-Pad1) -> GND
- C2 pad 2: GND -> /VBUS_3V3
- U2 pad 23: Net-(C2-Pad1) -> Net-(U2-Pad23)
- U2 pad 24: Net-(C3-Pad1) -> Net-(U2-Pad24)
- Y1 pad 1: Net-(C2-Pad1) -> /VBUS_3V3
- Y1 pad 2: Net-(C3-Pad1) -> GND
Routing:
- net (no net): track 0.00 -> 98.3 mm
- net GND: track 229.1 -> 177.3 mm
- net /VBUS_3V3: track 0.00 -> 10.7 mm
- net Net-(C2-Pad1): track 8.52 -> 0.00 mm
- net Net-(C3-Pad1): track 8.44 -> 0.00 mm
- net /VBUS: track 92.8 -> 97.1 mm
- net Net-(U2-Pad24): track 0.00 -> 4.30 mm
- net /Analog_out: track 18.2 -> 19.0 mm
- added copper zone on B.Cu, net GND
- added copper zone on F.Cu, net GND
Other:
- board text added: "GND"
- board text added: "VBUS"
